Commit message: ?

File: turtlebot_nonstop/turtlebot_nonstop_description/urdf/marker_bundle/marker_bundle_1.urdf.xacro (robot description, xacro)
@@ -38,8 +38,8 @@
   </xacro:macro>
   <xacro:macro name="marker_bundle_1" params="parent">
-    <attached_marker parent="${parent}" marker_num="4" direction="front" x_loc= "0.1" y_loc= "0" z_loc="0.5" r_deg="0" p_deg="1.570795" y_deg="0"/>
-    <attached_marker parent="${parent}" marker_num="5" direction="backward" x_loc= "-0.1" y_loc= "0" z_loc=".5" r_deg="3.14159" p_deg="1.570795" y_deg="0"/>
-    <attached_marker parent="${parent}" marker_num="6" direction="left" x_loc="0" y_loc= "-0.1" z_loc="0.5" r_deg="3.14159" p_deg="1.570795" y_deg="1.570795"/>
-    <attached_marker parent="${parent}" marker_num="7" direction="right" x_loc= "0" y_loc="0.1" z_loc="0.5" r_deg="0" p_deg="1.570795" y_deg="1.570795"/>
-      </xacro:macro>
+    <attached_marker parent="${parent}" marker_num="7" direction="front" x_loc= "0.08" y_loc= "0.08" z_loc="0.253" r_deg="0" p_deg="1.570795" y_deg="0"/>
+    <attached_marker parent="${parent}" marker_num="8" direction="backward" x_loc= "-0.16" y_loc= "0" z_loc="0.253" r_deg="3.14159" p_deg="1.570795" y_deg="0"/>
+    <attached_marker parent="${parent}" marker_num="9" direction="left" x_loc="0" y_loc= "-0.16" z_loc="0.253" r_deg="3.14159" p_deg="1.570795" y_deg="1.570795"/>
+    <attached_marker parent="${parent}" marker_num="10" direction="right" x_loc= "0" y_loc="0.16" z_loc="0.253" r_deg="0" p_deg="1.570795" y_deg="1.570795"/>
+  </xacro:macro>
 </robot>
