Commit message: frame

File: lemonabot/lemonabot_description/urdf/frame/lemonabot_frame.urdf.xacro (robot description, xacro)
@@ -1,11 +1,11 @@
 <?xml version="1.0"?>
 <robot name="lemonabot_frame" xmlns:xacro="http://ros.org/wiki/xacro">
-  <xacro:include filename="$(find lemonabot_description)/urdf/common_properties.urdf.xacro"/>
+  <xacro:include filename="$(find coldeyes_description)/urdf/common_properties.urdf.xacro"/>
   <link name="base_link">
     <visual>
       <geometry>
-        <box size=".50 .72 .29"/>
+        <box size=".38 .48 .36"/>
       </geometry>
-      <origin rpy="0 0 0" xyz="0 0 .145"/>
+      <origin rpy="0 0 0" xyz="0 0 .18"/>
       <material name="red">
         <color rgba=".8 0 0 1"/>
@@ -13,3 +13,38 @@
     </visual>
   </link>
+  <link name="bottom_plate_link">
+    <visual>
+      <geometry><link name="base_link">
+    <visual>
+      <geometry>
+        <box size=".38 .48 .002"/>
+      </geometry>
+      <origin rpy="0 0 0" xyz="0 0 0.03"/>
+      <material name="blue">
+        <color rgba="0 0 1 1"/>
+      </material>
+    </visual>
+  </link>
+  <link name="middle_plate_link">
+    <visual>
+      <geometry>
+        <box size=".38 .38 .002"/>
+      </geometry>
+      <origin rpy="0 0 0" xyz="0 0 .16"/>
+      <material name="green">
+        <color rgba="0 1 0 1"/>
+      </material>
+    </visual>
+  </link>
+  <link name="top_plate_link">
+    <visual>
+      <geometry>
+        <box size=".38 .38 .002"/>
+      </geometry>
+      <origin rpy="0 0 0" xyz="0 0 .245"/>
+      <material name="purple">
+        <color rgba="1 0 1 1"/>
+      </material>
+    </visual>
+  </link>
 </robot>

Commit message: frame_

File: lemonabot/lemonabot_description/urdf/frame/lemonabot_frame.urdf.xacro (robot description, xacro)
@@ -48,3 +48,14 @@
     </visual>
   </link>
+  <link name="hokuyo_link">
+    <visual>
+      <geometry>
+        <box size=".05 .05 .08"/>
+      </geometry>
+      <origin rpy="0 0 0" xyz="0.1 0 .29"/>
+      <material name="yellow">
+        <color rgba="1 1 1 0"/>
+      </material>
+    </visual>
+  </link>
 </robot>

File: lemonabot/lemonabot_description/urdf/marker_bundle/marker_bundle.urdf.xacro (robot description, xacro)
@@ -38,5 +38,5 @@
   </xacro:macro>
   <xacro:macro name="marker_bundle_0" params="parent">
-    <attached_marker parent="${parent}" marker_num="0" direction="front" x_loc= "0.19" y_loc= "0.19" z_loc="0.21" r_deg="0" p_deg="1.570795" y_deg="0"/>
+    <attached_marker parent="${parent}" marker_num="0" direction="front" x_loc= "0.19" y_loc= "0" z_loc="0.21" r_deg="0" p_deg="1.570795" y_deg="0"/>
     <attached_marker parent="${parent}" marker_num="1" direction="backward" x_loc= "-0.19" y_loc= "0" z_loc="0.21" r_deg="3.14159" p_deg="1.570795" y_deg="0"/>
     <attached_marker parent="${parent}" marker_num="2" direction="left" x_loc="0" y_loc= "-0.19" z_loc="0.21" r_deg="3.14159" p_deg="1.570795" y_deg="1.570795"/>

Commit message: frame

File: lemonabot/lemonabot_description/urdf/frame/lemonabot_frame.urdf.xacro (robot description, xacro)
@@ -48,14 +48,3 @@
     </visual>
   </link>
-  <link name="hokuyo_link">
-    <visual>
-      <geometry>
-        <box size=".05 .05 .08"/>
-      </geometry>
-      <origin rpy="0 0 0" xyz="0.1 0 .29"/>
-      <material name="yellow">
-        <color rgba="1 1 1 0"/>
-      </material>
-    </visual>
-  </link>
 </robot>

Commit message: frame

File: lemonabot/lemonabot_description/urdf/frame/lemonabot_frame.urdf.xacro (robot description, xacro)
@@ -14,6 +14,4 @@
   </link>
   <link name="bottom_plate_link">
-    <visual>
-      <geometry><link name="base_link">
     <visual>
       <geometry>

Commit message: joint

File: lemonabot/lemonabot_description/urdf/frame/lemonabot_frame.urdf.xacro (robot description, xacro)
@@ -2,4 +2,10 @@
 <robot name="lemonabot_frame" xmlns:xacro="http://ros.org/wiki/xacro">
   <xacro:include filename="$(find lemonabot_description)/urdf/common_properties.urdf.xacro"/>
+  <link name="base_footprint"/>
+  <joint name="base_joint" type="fixed">
+      <origin xyz="0 0 0" rpy="0 0 0" />
+      <parent link="base_footprint"/>
+      <child link="base_link" />
+  </joint>
   <link name="base_link">
     <visual>
@@ -13,4 +19,9 @@
     </visual>
   </link>
+  <joint name="bottom_plate_joint" type="fixed">
+      <origin xyz="0 0 0.03" rpy="0 0 0" />
+      <parent link="base_link"/>
+      <child link="bottom_plate_link" />
+  </joint>
   <link name="bottom_plate_link">
     <visual>
@@ -18,5 +29,5 @@
         <box size=".38 .48 .002"/>
       </geometry>
-      <origin rpy="0 0 0" xyz="0 0 0.03"/>
+      <origin rpy="0 0 0" xyz="0 0 0"/>
       <material name="blue">
         <color rgba="0 0 1 1"/>
@@ -24,4 +35,9 @@
     </visual>
   </link>
+  <joint name="middle_plate_joint" type="fixed">
+      <origin xyz="0 0 0.16" rpy="0 0 0" />
+      <parent link="base_link"/>
+      <child link="middle_plate_link" />
+  </joint>
   <link name="middle_plate_link">
     <visual>
@@ -29,5 +45,5 @@
         <box size=".38 .38 .002"/>
       </geometry>
-      <origin rpy="0 0 0" xyz="0 0 .16"/>
+      <origin rpy="0 0 0" xyz="0 0 0"/>
       <material name="green">
         <color rgba="0 1 0 1"/>
@@ -35,4 +51,9 @@
     </visual>
   </link>
+  <joint name="top_plate_joint" type="fixed">
+      <origin xyz="0 0 0.245" rpy="0 0 0" />
+      <parent link="base_link"/>
+      <child link="top_plate_link" />
+  </joint>
   <link name="top_plate_link">
     <visual>
@@ -40,5 +61,5 @@
         <box size=".38 .38 .002"/>
       </geometry>
-      <origin rpy="0 0 0" xyz="0 0 .245"/>
+      <origin rpy="0 0 0" xyz="0 0 0"/>
       <material name="purple">
         <color rgba="1 0 1 1"/>

Commit message: box X

File: lemonabot/lemonabot_description/urdf/frame/lemonabot_frame.urdf.xacro (robot description, xacro)
@@ -15,5 +15,5 @@
       <origin rpy="0 0 0" xyz="0 0 .18"/>
       <material name="red">
-        <color rgba=".8 0 0 1"/>
+        <color rgba="0.1 0 0 1"/>
       </material>
     </visual>
@@ -27,5 +27,6 @@
     <visual>
       <geometry>
-        <box size=".38 .48 .002"/>
+        <cylinder length="0.002" radius="0.19"/>
+       <!-- <box size=".38 .48 .002"/>-->
       </geometry>
       <origin rpy="0 0 0" xyz="0 0 0"/>
@@ -43,5 +44,6 @@
     <visual>
       <geometry>
-        <box size=".38 .38 .002"/>
+	<cylinder length="0.002" radius="0.19"/>
+        <!--<box size=".38 .38 .002"/>-->
       </geometry>
       <origin rpy="0 0 0" xyz="0 0 0"/>
@@ -59,5 +61,6 @@
     <visual>
       <geometry>
-        <box size=".38 .38 .002"/>
+	<cylinder length="0.002" radius="0.19"/>
+        <!--<box size=".38 .38 .002"/>-->
       </geometry>
       <origin rpy="0 0 0" xyz="0 0 0"/>

Commit message: body fin

File: lemonabot/lemonabot_description/urdf/frame/lemonabot_frame.urdf.xacro (robot description, xacro)
@@ -10,7 +10,4 @@
   <link name="base_link">
     <visual>
-      <geometry>
-        <box size=".38 .48 .36"/>
-      </geometry>
       <origin rpy="0 0 0" xyz="0 0 .18"/>
       <material name="red">

Commit message: wheel

File: lemonabot/lemonabot_description/urdf/frame/lemonabot_frame.urdf.xacro (robot description, xacro)
@@ -10,5 +10,5 @@
   <link name="base_link">
     <visual>
-      <origin rpy="0 0 0" xyz="0 0 .18"/>
+      <origin rpy="0 0 0" xyz="0 0 0"/>
       <material name="red">
         <color rgba="0.1 0 0 1"/>
@@ -28,6 +28,6 @@
       </geometry>
       <origin rpy="0 0 0" xyz="0 0 0"/>
-      <material name="blue">
-        <color rgba="0 0 1 1"/>
+      <material name="white">
+        <color rgba="0.9 1 1 1"/>
       </material>
     </visual>
@@ -45,6 +45,6 @@
       </geometry>
       <origin rpy="0 0 0" xyz="0 0 0"/>
-      <material name="green">
-        <color rgba="0 1 0 1"/>
+      <material name="white">
+        <color rgba="0.9 1 1 1"/>
       </material>
     </visual>
@@ -62,6 +62,41 @@
       </geometry>
       <origin rpy="0 0 0" xyz="0 0 0"/>
-      <material name="purple">
-        <color rgba="1 0 1 1"/>
+      <material name="white">
+        <color rgba="0.9 1 1 1"/>
+      </material>
+    </visual>
+  </link>
+  <!-- wheel -->
+  <joint name="left_wheel_joint" type="fixed">
+      <origin xyz="0 0.10 0" rpy="1.57075 1.57075 0" />
+      <parent link="bottom_plate_link"/>
+      <child link="left_wheel_link" />
+  </joint>
+  <link name="left_wheel_link">
+    <visual>
+      <geometry>
+        <cylinder length="0.02" radius="0.03"/>
+        <!--<box size=".38 .38 .002"/>-->
+      </geometry>
+      <origin rpy="0 0 0" xyz="0 0 0"/>
+      <material name="red">
+        <color rgba="1 0 0 1"/>
+      </material>
+    </visual>
+  </link>
+  <joint name="right_wheel_joint" type="fixed">
+      <origin xyz="0 -0.10 0" rpy="1.57075 1.57075 0" />
+      <parent link="bottom_plate_link"/>
+      <child link="right_wheel_link" />
+  </joint>
+  <link name="right_wheel_link">
+    <visual>
+      <geometry>
+        <cylinder length="0.02" radius="0.03"/>
+        <!--<box size=".38 .38 .002"/>-->
+      </geometry>
+      <origin rpy="0 0 0" xyz="0 0 0"/>
+      <material name="red">
+        <color rgba="1 0 0 1"/>
       </material>
     </visual>

Commit message: upload

File: lemonabot/lemonabot_description/urdf/frame/lemonabot_frame.urdf.xacro (robot description, xacro)
@@ -10,7 +10,10 @@
   <link name="base_link">
     <visual>
+      <geometry>
+        <box size=".38 .48 .002"/>
+      </geometry>
       <origin rpy="0 0 0" xyz="0 0 0"/>
       <material name="red">
-        <color rgba="0.1 0 0 1"/>
+        <color rgba="0 0 0 0"/>
       </material>
     </visual>
