Commit message: fix mapping

File: handheld_mappper/handheld_mapper_description/robots/handheld_mapper.urdf.xacro (robot description, xacro)
@@ -1,5 +1,16 @@
 <?xml version="1.0"?>
-<robot name="handheld_mapper" xmlns:xacro="http://ros.org/wiki/xacro">
+<robot xmlns:xacro="http://ros.org/wiki/xacro">
   <xacro:include filename="$(find handheld_mapper_description)/urdf/handheld_mapper_library.urdf.xacro" />
-  <handheld_mapper/>
+    <link name="base_link">
+    <visual>
+      <geometry>
+        <box size=".38 .48 .36"/>
+      </geometry>
+      <origin rpy="0 0 0" xyz="0 0 .18"/>
+      <material name="red">
+        <color rgba=".8 0 0 1"/>
+      </material>
+    </visual>
+  </link>
+  <handheld_mapper parent="base_link" x_loc="0.10" y_loc="0.0" z_loc="0.245" r_deg="0.0" p_deg="0.0" y_deg="0.0"/>
 </robot>

File: handheld_mappper/handheld_mapper_description/urdf/handheld_mapper.urdf.xacro (robot description, xacro)
@@ -1,15 +1,12 @@
 <?xml version="1.0"?>
-<root xmlns:xacro="http://ros.org/wiki/xacro">
+<robot name="handheld_mapper" xmlns:xacro="http://ros.org/wiki/xacro">
   <!-- Included URDF Files -->
-  <xacro:include filename="$(find handheld_mapper_description)/urdf/common_properties.urdf.xacro"/>
-  <xacro:macro name="handheld_mapper">
-  <link name="base_footprint">
-    <joint name="base_joint" type="fixed">
-      <origin xyz="0 0 0.0015" rpy="0 0 0" />
-      <parent link="base_footprint"/>
-      <child link="base_link" />
-    </joint>
-  </link>
-  <link name="base_link">
+  <xacro:macro name="handheld_mapper" params="parent x_loc y_loc z_loc r_deg p_deg y_deg">
+  <joint name="handheld_mapper_joint" type="fixed">
+      <origin xyz="${x_loc} ${y_loc} ${z_loc}" rpy="${r_deg} ${p_deg} ${y_deg}"/>
+      <parent link="${parent}"/>
+      <child link="laser_base_link"/>
+  </joint>
+  <link name="laser_base_link">
     <visual>
       <geometry>
@@ -17,16 +14,13 @@
       </geometry>
       <origin rpy="0 0 0" xyz="0 0 .18"/>
-      <material name="red">
-        <color rgba=".8 0 0 1"/>
-      </material>
     </visual>
   </link>
   <!-- laser -->
-    <xacro:hokuyo_04lx_laser name="hokuyo" parent="base">
+    <xacro:hokuyo_04lx_laser name="hokuyo" parent="laser_base">
       <origin xyz="-0.075 0 0.003" rpy="0 0 0" />
     </xacro:hokuyo_04lx_laser>
     <!-- imu -->
     <joint name="base_to_imu" type="fixed">
-      <parent link="base_link"/>
+      <parent link="laser_base_link"/>
       <child link="imu"/>
       <origin xyz="0.075 0.01 0.04"/>
@@ -38,7 +32,6 @@
         </geometry>
         <origin rpy="0 0 0" xyz="0 0 0"/>
-        <material name="white"/>
       </visual>
     </link>
   </xacro:macro>
-</root>
+</robot>

File: handheld_mappper/handheld_mapper_description/urdf/handheld_mapper_library.urdf.xacro (robot description, xacro)
@@ -4,11 +4,9 @@
  -->
 <robot xmlns:xacro="http://ros.org/wiki/xacro">
-  <!-- General -->
-  <xacro:include filename="$(find handheld_mapper_description)/urdf/common.urdf.xacro"/>
+  <!-- General
+  <xacro:include filename="$(find handheld_mapper_description)/urdf/common.urdf.xacro"/>-->
   <!-- Laser Sensors -->
   <xacro:include filename="$(find handheld_mapper_description)/urdf/sensors/hokuyo_04lx_laser.urdf.xacro"/>
   <!-- Stack -->
   <xacro:include filename="$(find handheld_mapper_description)/urdf/handheld_mapper.urdf.xacro"/>
- <!-- Bundle Markers -->
-  <xacro:include filename="$(find handheld_mapper_description)/urdf/marker_bundle/marker_bundle.urdf.xacro"/>
 </robot>

File: lemonabot/lemonabot_description/urdf/lemonabot_library.urdf.xacro (robot description, xacro)
@@ -1,20 +1,7 @@
 <?xml version="1.0"?>
-<!--
-  The complete turtlebot library of xacros for easy reference
- -->
 <robot xmlns:xacro="http://ros.org/wiki/xacro">
-  <!-- General -->
-  <!--<xacro:include filename="$(find turtlebot_nonstop_description)/urdf/common_properties.urdf.xacro"/>
-  <xacro:include filename="$(find turtlebot_nonstop_description)/urdf/turtlebot_properties.urdf.xacro"/>
-  <!-- Bases -->
-  <!--<xacro:include filename="$(find kobuki_description)/urdf/kobuki.urdf.xacro" />
-  <!-- Stacks -->
-  <!--<xacro:include filename="$(find turtlebot_nonstop_description)/urdf/stacks/circles.urdf.xacro"/>
-  <xacro:include filename="$(find turtlebot_nonstop_description)/urdf/stacks/hexagons.urdf.xacro"/>
-  <!-- 3D Sensors -->
-  <!--<xacro:include filename="$(find turtlebot_nonstop_description)/urdf/sensors/kinect.urdf.xacro"/>
+  <xacro:include filename="$(find lemonabot_description)/urdf/frame/lemonabot_frame.urdf.xacro"/>
+  <xacro:include filename="$(find handheld_mapper_description)/urdf/handheld_mapper_library.urdf.xacro"/>
   <!-- Bundle Markers -->
   <xacro:include filename="$(find lemonabot_description)/urdf/marker_bundle/marker_bundle.urdf.xacro"/>
 </robot>
-~
-~

Commit message: filename

File: handheld_mappper/handheld_mapper_description/robots/handheld_mapper.urdf.xacro (robot description, xacro)
@@ -2,12 +2,18 @@
 <robot name="handheld_mapperbot" xmlns:xacro="http://ros.org/wiki/xacro">
   <xacro:include filename="$(find handheld_mapper_description)/urdf/handheld_mapper_library.urdf.xacro" />
-    <link name="base_link">
+  <link name="base_footprint"/>
+  <joint name="base_joint" type="fixed">
+      <origin xyz="0 0 0" rpy="0 0 0" />
+      <parent link="base_footprint"/>
+      <child link="base_link" />
+  </joint>
+  <link name="base_link">
     <visual>
       <geometry>
-        <box size=".38 .48 .36"/>
+        <box size=".38 .48 .002"/>
       </geometry>
-      <origin rpy="0 0 0" xyz="0 0 .18"/>
+      <origin rpy="0 0 0" xyz="0 0 0"/>
       <material name="red">
-        <color rgba=".8 0 0 1"/>
+        <color rgba="0 0 0 0"/>
       </material>
     </visual>
