Commit message: odom

File: handheld_mappper/handheld_mapper_description/urdf/handheld_mapper.urdf.xacro (robot description, xacro)
@@ -5,4 +5,10 @@
   <xacro:include filename="$(find handheld_mapper_description)/urdf/common_properties.urdf.xacro"/>
   <xacro:macro name="handheld_mapper">
+<link name="base_footprint"/>
+    <joint name="base_joint" type="fixed">
+      <origin xyz="0 0 0.0015" rpy="0 0 0" />
+      <parent link="base_footprint"/>
+      <child link="base_link" />
+    </joint>
     <link name="base_link">
       <visual>

Commit message: _

File: handheld_mappper/handheld_mapper_description/urdf/handheld_mapper.urdf.xacro (robot description, xacro)
@@ -5,5 +5,5 @@
   <xacro:include filename="$(find handheld_mapper_description)/urdf/common_properties.urdf.xacro"/>
   <xacro:macro name="handheld_mapper">
-<link name="base_footprint"/>
+  <link name="base_footprint"/>
     <joint name="base_joint" type="fixed">
       <origin xyz="0 0 0.0015" rpy="0 0 0" />
@@ -11,14 +11,63 @@
       <child link="base_link" />
     </joint>
-    <link name="base_link">
-      <visual>
-        <origin xyz="0 0 0" rpy="0 0 0" />
-        <geometry>
-          <box size="0.26 0.18 0.03"/>
-        </geometry>
-        <material name="white"/>
-      </visual>
-    </link>
-    <!-- laser -->
+  </link>
+  <link name="base_link">
+    <visual>
+      <geometry>
+        <box size=".38 .48 .36"/>
+      </geometry>
+      <origin rpy="0 0 0" xyz="0 0 .18"/>
+      <material name="red">
+        <color rgba=".8 0 0 1"/>
+      </material>
+    </visual>
+  </link>
+  <link name="bottom_plate_link">
+    <visual>
+      <geometry><link name="base_link">
+    <visual>
+      <geometry>
+        <box size=".38 .48 .002"/>
+      </geometry>
+      <origin rpy="0 0 0" xyz="0 0 0.03"/>
+      <material name="blue">
+        <color rgba="0 0 1 1"/>
+      </material>
+    </visual>
+  </link>
+  <link name="middle_plate_link">
+    <visual>
+      <geometry>
+        <box size=".38 .38 .002"/>
+      </geometry>
+      <origin rpy="0 0 0" xyz="0 0 .16"/>
+      <material name="green">
+        <color rgba="0 1 0 1"/>
+      </material>
+    </visual>
+  </link>
+  <link name="top_plate_link">
+    <visual>
+      <geometry>
+        <box size=".38 .38 .002"/>
+      </geometry>
+      <origin rpy="0 0 0" xyz="0 0 .245"/>
+      <material name="purple">
+        <color rgba="1 0 1 1"/>
+      </material>
+    </visual>
+  </link>
+  <link name="battery_link">
+    <visual>
+      <geometry>
+        <box size=".15 .085 .1"/>
+      </geometry>
+      <origin rpy="0 0 0" xyz="0 0 .295"/>
+      <material name="cobalt">
+        <color rgba="0 0 .5 1"/>
+      </material>
+    </visual>
+  </link>
+  <!-- laser -->
     <xacro:hokuyo_04lx_laser name="hokuyo" parent="base">
       <origin xyz="-0.075 0 0.003" rpy="0 0 0" />

File: lemonabot/lemonabot_description/urdf/frame/lemonabot_frame.urdf.xacro (robot description, xacro)
@@ -5,7 +5,7 @@
     <visual>
       <geometry>
-        <box size=".38 .48 .36"/>
+        <box size=".50 .72 .29"/>
       </geometry>
-      <origin rpy="0 0 0" xyz="0 0 .18"/>
+      <origin rpy="0 0 0" xyz="0 0 .145"/>
       <material name="red">
         <color rgba=".8 0 0 1"/>
@@ -13,60 +13,3 @@
     </visual>
   </link>
-  <link name="bottom_plate_link">
-    <visual>
-      <geometry><link name="base_link">
-    <visual>
-      <geometry>
-        <box size=".38 .48 .002"/>
-      </geometry>
-      <origin rpy="0 0 0" xyz="0 0 0.03"/>
-      <material name="blue">
-        <color rgba="0 0 1 1"/>
-      </material>
-    </visual>
-  </link>
-  <link name="middle_plate_link">
-    <visual>
-      <geometry>
-        <box size=".38 .38 .002"/>
-      </geometry>
-      <origin rpy="0 0 0" xyz="0 0 .16"/>
-      <material name="green">
-        <color rgba="0 1 0 1"/>
-      </material>
-    </visual>
-  </link>
-  <link name="top_plate_link">
-    <visual>
-      <geometry>
-        <box size=".38 .38 .002"/>
-      </geometry>
-      <origin rpy="0 0 0" xyz="0 0 .245"/>
-      <material name="purple">
-        <color rgba="1 0 1 1"/>
-      </material>
-    </visual>
-  </link>
-  <link name="battery_link">
-    <visual>
-      <geometry>
-        <box size=".15 .085 .1"/>
-      </geometry>
-      <origin rpy="0 0 0" xyz="0 0 .295"/>
-      <material name="cobalt">
-        <color rgba="0 0 .5 1"/>
-      </material>
-    </visual>
-  </link>
-  <link name="gun_base_link">
-    <visual>
-      <geometry>
-        <box size=".05 .05 .05"/>
-      </geometry>
-      <origin rpy="0 0 0" xyz="0 0.13 .325"/>
-      <material name="teal">
-        <color rgba="0 1 1 1"/>
-      </material>
-    </visual>
-  </link>
 </robot>

File: sniperbot/sniperbot_description/urdf/sniperbot_library.urdf.xacro (robot description, xacro)
@@ -15,5 +15,5 @@
   <!--<xacro:include filename="$(find turtlebot_nonstop_description)/urdf/sensors/kinect.urdf.xacro"/>
   <!-- Bundle Markers -->
-  <xacro:include filename="$(find lemonabot_description)/urdf/marker_bundle/marker_bundle.urdf.xacro"/>
+  <xacro:include filename="$(find sniperbot_description)/urdf/marker_bundle/marker_bundle.urdf.xacro"/>
 </robot>
 ~

Commit message: roll back

File: handheld_mappper/handheld_mapper_description/urdf/handheld_mapper.urdf.xacro (robot description, xacro)
@@ -23,50 +23,4 @@
     </visual>
   </link>
-  <link name="bottom_plate_link">
-    <visual>
-      <geometry><link name="base_link">
-    <visual>
-      <geometry>
-        <box size=".38 .48 .002"/>
-      </geometry>
-      <origin rpy="0 0 0" xyz="0 0 0.03"/>
-      <material name="blue">
-        <color rgba="0 0 1 1"/>
-      </material>
-    </visual>
-  </link>
-  <link name="middle_plate_link">
-    <visual>
-      <geometry>
-        <box size=".38 .38 .002"/>
-      </geometry>
-      <origin rpy="0 0 0" xyz="0 0 .16"/>
-      <material name="green">
-        <color rgba="0 1 0 1"/>
-      </material>
-    </visual>
-  </link>
-  <link name="top_plate_link">
-    <visual>
-      <geometry>
-        <box size=".38 .38 .002"/>
-      </geometry>
-      <origin rpy="0 0 0" xyz="0 0 .245"/>
-      <material name="purple">
-        <color rgba="1 0 1 1"/>
-      </material>
-    </visual>
-  </link>
-  <link name="battery_link">
-    <visual>
-      <geometry>
-        <box size=".15 .085 .1"/>
-      </geometry>
-      <origin rpy="0 0 0" xyz="0 0 .295"/>
-      <material name="cobalt">
-        <color rgba="0 0 .5 1"/>
-      </material>
-    </visual>
-  </link>
   <!-- laser -->
     <xacro:hokuyo_04lx_laser name="hokuyo" parent="base">

Commit message: modified urdf files

File: handheld_mappper/handheld_mapper_description/urdf/handheld_mapper.urdf.xacro (robot description, xacro)
@@ -14,4 +14,7 @@
       </geometry>
       <origin rpy="0 0 0" xyz="0 0 .18"/>
+      <material name="red">
+        <color rgba="0 0 0 0"/>
+      </material>
     </visual>
   </link>
@@ -32,4 +35,7 @@
         </geometry>
         <origin rpy="0 0 0" xyz="0 0 0"/>
+      <material name="black">
+        <color rgba="0 0 0 1"/>
+      </material>
       </visual>
     </link>

File: handheld_mappper/handheld_mapper_description/urdf/handheld_mapper_library.urdf.xacro (robot description, xacro)
@@ -3,5 +3,5 @@
   The complete handheld_mapper library of xacros for easy reference
  -->
-<robot xmlns:xacro="http://ros.org/wiki/xacro">
+<robot name="handheld" xmlns:xacro="http://ros.org/wiki/xacro">
   <!-- General
   <xacro:include filename="$(find handheld_mapper_description)/urdf/common.urdf.xacro"/>-->
