Commit message: resized marker

File: coldeyes/coldeyes_description/urdf/marker_bundle/marker_bundle.urdf.xacro (robot description, xacro)
@@ -15,5 +15,5 @@
         <origin xyz="0 0 0" rpy="0 0 0"/>
         <geometry>
-          <box size="0.04 0.04 0.001"/>
+          <box size="0.09 0.09 0.001"/>
         </geometry>
         <material name="am_${marker_num}">
