Commit message: modified urdf

File: lemonabot/lemonabot_description/robots/lemonabot.urdf.xacro (robot description, xacro)
@@ -3,3 +3,5 @@
   <xacro:include filename="$(find lemonabot_description)/urdf/lemonabot_library.urdf.xacro" />
   <lemonabot_frame/>
+  <marker_bundle_0 parent="base_link"/>
+  <handheld_mapper parent="base_link" x_loc="0.10" y_loc="0.0" z_loc="0.245" r_deg="0.0" p_deg="0.0" y_deg="0.0"/>
 </robot>

File: lemonabot/lemonabot_description/urdf/frame/lemonabot_frame.urdf.xacro (robot description, xacro)
@@ -14,5 +14,5 @@
       </geometry>
       <origin rpy="0 0 0" xyz="0 0 0"/>
-      <material name="red">
+      <material name="none">
         <color rgba="0 0 0 0"/>
       </material>
@@ -28,5 +28,4 @@
       <geometry>
         <cylinder length="0.002" radius="0.19"/>
-       <!-- <box size=".38 .48 .002"/>-->
       </geometry>
       <origin rpy="0 0 0" xyz="0 0 0"/>
@@ -45,5 +44,4 @@
       <geometry>
 	<cylinder length="0.002" radius="0.19"/>
-        <!--<box size=".38 .38 .002"/>-->
       </geometry>
       <origin rpy="0 0 0" xyz="0 0 0"/>
@@ -62,5 +60,4 @@
       <geometry>
 	<cylinder length="0.002" radius="0.19"/>
-        <!--<box size=".38 .38 .002"/>-->
       </geometry>
       <origin rpy="0 0 0" xyz="0 0 0"/>
@@ -72,5 +69,5 @@
   <!-- wheel -->
   <joint name="left_wheel_joint" type="fixed">
-      <origin xyz="0 0.10 0" rpy="1.57075 1.57075 0" />
+      <origin xyz="-0.04 0.10 0.03" rpy="1.57075 1.57075 0" />
       <parent link="bottom_plate_link"/>
       <child link="left_wheel_link" />
@@ -79,15 +76,14 @@
     <visual>
       <geometry>
-        <cylinder length="0.02" radius="0.03"/>
-        <!--<box size=".38 .38 .002"/>-->
+        <cylinder length="0.02" radius="0.06"/>
       </geometry>
       <origin rpy="0 0 0" xyz="0 0 0"/>
-      <material name="red">
-        <color rgba="1 0 0 1"/>
+      <material name="blood">
+        <color rgba="0.6 0 0 1"/>
       </material>
     </visual>
   </link>
   <joint name="right_wheel_joint" type="fixed">
-      <origin xyz="0 -0.10 0" rpy="1.57075 1.57075 0" />
+      <origin xyz="-0.04 -0.10 0.03" rpy="1.57075 1.57075 0" />
       <parent link="bottom_plate_link"/>
       <child link="right_wheel_link" />
@@ -96,10 +92,9 @@
     <visual>
       <geometry>
-        <cylinder length="0.02" radius="0.03"/>
-        <!--<box size=".38 .38 .002"/>-->
+        <cylinder length="0.02" radius="0.06"/>
       </geometry>
       <origin rpy="0 0 0" xyz="0 0 0"/>
-      <material name="red">
-        <color rgba="1 0 0 1"/>
+      <material name="blood">
+        <color rgba="0.6 0 0 1"/>
       </material>
     </visual>

File: lemonabot/lemonabot_description/urdf/marker_bundle/marker_bundle.urdf.xacro (robot description, xacro)
@@ -42,4 +42,4 @@
     <attached_marker parent="${parent}" marker_num="2" direction="left" x_loc="0" y_loc= "-0.19" z_loc="0.21" r_deg="3.14159" p_deg="1.570795" y_deg="1.570795"/>
     <attached_marker parent="${parent}" marker_num="3" direction="right" x_loc= "0" y_loc="0.19" z_loc="0.21" r_deg="0" p_deg="1.570795" y_deg="1.570795"/>
-      </xacro:macro>
+  </xacro:macro>
 </robot>

Commit message: lemon

File: lemonabot/lemonabot_description/robots/lemonabot.urdf.xacro (robot description, xacro)
@@ -4,4 +4,4 @@
   <lemonabot_frame/>
   <marker_bundle_0 parent="base_link"/>
-  <handheld_mapper parent="base_link" x_loc="0.10" y_loc="0.0" z_loc="0.245" r_deg="0.0" p_deg="0.0" y_deg="0.0"/>
+  <handheld_mapper parent="base_link" x_loc="0.10" y_loc="0.0" z_loc="0.247" r_deg="0.0" p_deg="0.0" y_deg="0.0"/>
 </robot>

File: lemonabot/lemonabot_description/urdf/frame/lemonabot_frame.urdf.xacro (robot description, xacro)
@@ -27,9 +27,9 @@
     <visual>
       <geometry>
-        <cylinder length="0.002" radius="0.19"/>
-      </geometry>
-      <origin rpy="0 0 0" xyz="0 0 0"/>
-      <material name="white">
-        <color rgba="0.9 1 1 1"/>
+        <cylinder length="0.002" radius="0.22"/>
+      </geometry>
+      <origin rpy="0 0 0" xyz="0 0 0"/>
+      <material name="plate_metal">
+        <color rgba="0.5 0.54 0.55 1"/>
       </material>
     </visual>
@@ -46,6 +46,6 @@
       </geometry>
       <origin rpy="0 0 0" xyz="0 0 0"/>
-      <material name="white">
-        <color rgba="0.9 1 1 1"/>
+      <material name="plate_white">
+        <color rgba="0.7 0.7 0.65 1"/>
       </material>
     </visual>
@@ -62,12 +62,26 @@
       </geometry>
       <origin rpy="0 0 0" xyz="0 0 0"/>
-      <material name="white">
-        <color rgba="0.9 1 1 1"/>
-      </material>
+      <material name="plate_white" />
     </visual>
   </link>
   <!-- wheel -->
+  <joint name="left_tire_joint" type="fixed">
+      <origin xyz="-0.06 0.12 0.035" rpy="1.57075 1.57075 0" />
+      <parent link="bottom_plate_link"/>
+      <child link="left_tire_link" />
+  </joint>
+  <link name="left_tire_link">
+    <visual>
+      <geometry>
+        <cylinder length="0.025" radius="0.065"/>
+      </geometry>
+      <origin rpy="0 0 0" xyz="0 0 0"/>
+      <material name="black">
+        <color rgba="0.2 0.2 0.2 1"/>
+      </material>
+    </visual>
+  </link>
   <joint name="left_wheel_joint" type="fixed">
-      <origin xyz="-0.04 0.10 0.03" rpy="1.57075 1.57075 0" />
+      <origin xyz="-0.06 0.12 0.035" rpy="1.57075 1.57075 0" />
       <parent link="bottom_plate_link"/>
       <child link="left_wheel_link" />
@@ -76,14 +90,28 @@
     <visual>
       <geometry>
-        <cylinder length="0.02" radius="0.06"/>
-      </geometry>
-      <origin rpy="0 0 0" xyz="0 0 0"/>
-      <material name="blood">
-        <color rgba="0.6 0 0 1"/>
-      </material>
+        <cylinder length="0.027" radius="0.05"/>
+      </geometry>
+      <origin rpy="0 0 0" xyz="0 0 0"/>
+      <material name="gray">
+        <color rgba="0.8 0.8 0.8 1"/>
+      </material>
+    </visual>
+  </link>
+  <joint name="right_tire_joint" type="fixed">
+      <origin xyz="-0.06 -0.12 0.035" rpy="1.57075 1.57075 0" />
+      <parent link="bottom_plate_link"/>
+      <child link="right_tire_link" />
+  </joint>
+  <link name="right_tire_link">
+    <visual>
+      <geometry>
+        <cylinder length="0.025" radius="0.065"/>
+      </geometry>
+      <origin rpy="0 0 0" xyz="0 0 0"/>
+      <material name="black" />
     </visual>
   </link>
   <joint name="right_wheel_joint" type="fixed">
-      <origin xyz="-0.04 -0.10 0.03" rpy="1.57075 1.57075 0" />
+      <origin xyz="-0.06 -0.12 0.035" rpy="1.57075 1.57075 0" />
       <parent link="bottom_plate_link"/>
       <child link="right_wheel_link" />
@@ -92,10 +120,125 @@
     <visual>
       <geometry>
-        <cylinder length="0.02" radius="0.06"/>
-      </geometry>
-      <origin rpy="0 0 0" xyz="0 0 0"/>
-      <material name="blood">
-        <color rgba="0.6 0 0 1"/>
-      </material>
+        <cylinder length="0.027" radius="0.05"/>
+      </geometry>
+      <origin rpy="0 0 0" xyz="0 0 0"/>
+      <material name="gray" />
+    </visual>
+  </link>
+  <!-- pole -->
+  <joint name="bottom_pole_1_joint" type="fixed">
+      <origin xyz="0.14 0.11 0.065" rpy="0 0 0" />
+      <parent link="bottom_plate_link"/>
+      <child link="bottom_pole_1_link" />
+  </joint>
+  <link name="bottom_pole_1_link">
+    <visual>
+      <geometry>
+        <cylinder length="0.13" radius="0.005"/>
+      </geometry>
+      <origin rpy="0 0 0" xyz="0 0 0"/>
+      <material name="gold">
+        <color rgba="0.55 0.5 0 1"/>
+      </material>
+    </visual>
+  </link>
+  <joint name="bottom_pole_2_joint" type="fixed">
+      <origin xyz="-0.14 0.11 0.065" rpy="0 0 0" />
+      <parent link="bottom_plate_link"/>
+      <child link="bottom_pole_2_link" />
+  </joint>
+  <link name="bottom_pole_2_link">
+    <visual>
+      <geometry>
+        <cylinder length="0.13" radius="0.005"/>
+      </geometry>
+      <origin rpy="0 0 0" xyz="0 0 0"/>
+      <material name="gold" />
+    </visual>
+  </link>
+  <joint name="bottom_pole_3_joint" type="fixed">
+      <origin xyz="-0.14 -0.11 0.065" rpy="0 0 0" />
+      <parent link="bottom_plate_link"/>
+      <child link="bottom_pole_3_link" />
+  </joint>
+  <link name="bottom_pole_3_link">
+    <visual>
+      <geometry>
+        <cylinder length="0.13" radius="0.005"/>
+      </geometry>
+      <origin rpy="0 0 0" xyz="0 0 0"/>
+      <material name="gold"/>
+    </visual>
+  </link>
+  <joint name="bottom_pole_4_joint" type="fixed">
+      <origin xyz="0.14 -0.11 0.065" rpy="0 0 0" />
+      <parent link="bottom_plate_link"/>
+      <child link="bottom_pole_4_link" />
+  </joint>
+  <link name="bottom_pole_4_link">
+    <visual>
+      <geometry>
+        <cylinder length="0.13" radius="0.005"/>
+      </geometry>
+      <origin rpy="0 0 0" xyz="0 0 0"/>
+      <material name="gold"/>
+    </visual>
+  </link>
+  <joint name="middle_pole_1_joint" type="fixed">
+      <origin xyz="0.12 0.12 0.043" rpy="0 0 0" />
+      <parent link="middle_plate_link"/>
+      <child link="middle_pole_1_link" />
+  </joint>
+  <link name="middle_pole_1_link">
+    <visual>
+      <geometry>
+        <cylinder length="0.085" radius="0.005"/>
+      </geometry>
+      <origin rpy="0 0 0" xyz="0 0 0"/>
+      <material name="gold"/>
+    </visual>
+  </link>
+  <joint name="middle_pole_2_joint" type="fixed">
+      <origin xyz="-0.12 0.12 0.043" rpy="0 0 0" />
+      <parent link="middle_plate_link"/>
+      <child link="middle_pole_2_link" />
+  </joint>
+  <link name="middle_pole_2_link">
+    <visual>
+      <geometry>
+        <cylinder length="0.085" radius="0.005"/>
+      </geometry>
+  <material name="black">
+        <color rgba="0.2 0.2 0.2 1"/>
+      </material>    <origin rpy="0 0 0" xyz="0 0 0"/>
+      <material name="gold"/>
+    </visual>
+  </link>
+  <joint name="middle_pole_3_joint" type="fixed">
+      <origin xyz="-0.12 -0.12 0.043" rpy="0 0 0" />
+      <parent link="middle_plate_link"/>
+      <child link="middle_pole_3_link" />
+  </joint>
+  <link name="middle_pole_3_link">
+    <visual>
+      <geometry>
+        <cylinder length="0.085" radius="0.005"/>
+      </geometry>
+      <origin rpy="0 0 0" xyz="0 0 0"/>
+      <material name="gold"/>
+    </visual>
+  </link>
+  <joint name="middle_pole_4_joint" type="fixed">
+      <origin xyz="0.12 -0.12 0.043" rpy="0 0 0" />
+      <parent link="middle_plate_link"/>
+      <child link="middle_pole_4_link" />
+  </joint>
+  <link name="middle_pole_4_link">
+    <visual>
+      <geometry>
+        <cylinder length="0.085" radius="0.005"/>
+      </geometry>
+      <origin rpy="0 0 0" xyz="0 0 0"/>
+      <material name="gold"/>
     </visual>
   </link>
