Commit message: +backward cam

File: coldeyes/coldeyes_description/urdf/frame/coldeyes_frame.urdf.xacro (robot description, xacro)
@@ -16,9 +16,20 @@
     <visual>
       <geometry>
+        <box size=".01 .01 .02"/>
+      </geometry>
+      <origin rpy="-1.57075 0 3.141592" xyz="0 0 0"/>
+      <material name="blue">
+        <color rgba="0 0 1 1"/>
+      </material>
+    </visual>
+  </link>
+  <link name="camera_backward">
+    <visual>
+      <geometry>
         <box size=".09 .01 .02"/>
       </geometry>
       <origin rpy="1.57075 0 0" xyz="0 0 0"/>
-      <material name="blue">
-        <color rgba="0 0 1 1"/>
+      <material name="green">
+        <color rgba="0 1 0 1"/>
       </material>
     </visual>

Commit message: clean

File: coldeyes/coldeyes_description/urdf/frame/coldeyes_frame.urdf.xacro (robot description, xacro)
@@ -24,4 +24,9 @@
     </visual>
   </link>
+  <joint name="base_to_camera_front" type="fixed">
+    <parent link="base_link"/>
+    <child link="camera_front"/>
+    <origin rpy="-1.57075 0 0" xyz="0 .0205 0.53"/>
+  </joint>
   <link name="camera_backward">
     <visual>
@@ -35,8 +40,8 @@
     </visual>
   </link>
-  <joint name="base_to_camera_front" type="fixed">
+  <joint name="base_to_camera_backward" type="fixed">
     <parent link="base_link"/>
-    <child link="camera_front"/>
-    <origin rpy="-1.57075 0 0" xyz="0 .0205 0.53"/>
+    <child link="camera_backward"/>
+    <origin rpy="1.57075 0 0" xyz="0 -0.0205 0.53"/>
   </joint>
   <link name="x_leg">

Commit message: hydro fetch

File: coldeyes/coldeyes_description/urdf/frame/coldeyes_frame.urdf.xacro (robot description, xacro)
@@ -16,7 +16,7 @@
     <visual>
       <geometry>
-        <box size=".01 .01 .02"/>
+        <box size=".01 .09 .02 "/>
       </geometry>
-      <origin rpy="-1.57075 0 3.141592" xyz="0 0 0"/>
+      <origin rpy="0 0 0" xyz="0 0 0"/>
       <material name="blue">
         <color rgba="0 0 1 1"/>
@@ -27,12 +27,13 @@
     <parent link="base_link"/>
     <child link="camera_front"/>
-    <origin rpy="-1.57075 0 0" xyz="0 .0205 0.53"/>
+    <origin rpy="3.141592 0 0" xyz=".0205 0 0.53"/>
   </joint>
+<!--
   <link name="camera_backward">
     <visual>
       <geometry>
-        <box size=".09 .01 .02"/>
+        <box size=".01 .01 .02"/>
       </geometry>
-      <origin rpy="1.57075 0 0" xyz="0 0 0"/>
+      <origin rpy="3.141592 0 0" xyz="0 0 0"/>
       <material name="green">
         <color rgba="0 1 0 1"/>
@@ -43,6 +44,7 @@
     <parent link="base_link"/>
     <child link="camera_backward"/>
-    <origin rpy="1.57075 0 0" xyz="0 -0.0205 0.53"/>
+    <origin rpy="0 0 0" xyz="0 -0.0205 0.53"/>
   </joint>
+-->
   <link name="x_leg">
     <visual>

Commit message: mapper

File: coldeyes/coldeyes_description/urdf/frame/coldeyes_frame.urdf.xacro (robot description, xacro)
@@ -27,5 +27,5 @@
     <parent link="base_link"/>
     <child link="camera_front"/>
-    <origin rpy="3.141592 0 0" xyz=".0205 0 0.53"/>
+    <origin rpy="-1.57075 0 -1.57075" xyz=".0205 0 0.53"/>
   </joint>
 <!--

File: handheld_mappper/handheld_mapper_description/urdf/handheld_mapper.urdf.xacro (robot description, xacro)
@@ -1,9 +1,8 @@
 <?xml version="1.0"?>
-<root
-      xmlns:xacro="http://ros.org/wiki/xacro">
+<root xmlns:xacro="http://ros.org/wiki/xacro">
   <!-- Included URDF Files -->
   <xacro:include filename="$(find handheld_mapper_description)/urdf/common_properties.urdf.xacro"/>
   <xacro:macro name="handheld_mapper">
-  <link name="base_footprint"/>
+  <link name="base_footprint">
     <joint name="base_joint" type="fixed">
       <origin xyz="0 0 0.0015" rpy="0 0 0" />

Commit message: up

File: coldeyes/coldeyes_description/urdf/frame/coldeyes_frame.urdf.xacro (robot description, xacro)
@@ -16,5 +16,5 @@
     <visual>
       <geometry>
-        <box size=".01 .09 .02 "/>
+        <box size=".09 .02 .01 "/>
       </geometry>
       <origin rpy="0 0 0" xyz="0 0 0"/>

Commit message: marker direction

File: coldeyes/coldeyes_description/urdf/frame/coldeyes_frame.urdf.xacro (robot description, xacro)
@@ -5,7 +5,7 @@
     <visual>
       <geometry>
-        <box size=".03 .03 .54"/>
+        <box size=".03 .03 .25"/>
       </geometry>
-      <origin rpy="0 0 0" xyz="0 0 .280"/>
+      <origin rpy="0 0 0" xyz="0 0 .140"/>
       <material name="red">
         <color rgba=".8 0 0 1"/>
@@ -27,5 +27,5 @@
     <parent link="base_link"/>
     <child link="camera_front"/>
-    <origin rpy="-1.57075 0 -1.57075" xyz=".0205 0 0.53"/>
+    <origin rpy="-1.57075 0 -1.57075" xyz=".0205 0 0.26"/>
   </joint>
 <!--

File: coldeyes/coldeyes_description/urdf/marker_bundle/marker_bundle.urdf.xacro (robot description, xacro)
@@ -37,6 +37,6 @@
   </xacro:macro>
   <xacro:macro name="marker_bundle" params="parent">
-    <attached_marker parent="${parent}" marker_num="0" direction="front" x_loc="0.015" y_loc= "0" z_loc="0.3" r_deg="1.570795" p_deg="1.570795" y_deg="1.570795"/>
-    <attached_marker parent="${parent}" marker_num="1" direction="back" x_loc= "-0.015" y_loc="0" z_loc="0.3" r_deg="-1.570795" p_deg="1.570795" y_deg="1.570795"/>
+    <attached_marker parent="${parent}" marker_num="0" direction="front" x_loc="0.015" y_loc= "0" z_loc="0.1" r_deg="1.570795" p_deg="1.570795" y_deg="1.570795"/>
+    <attached_marker parent="${parent}" marker_num="1" direction="back" x_loc= "-0.015" y_loc="0" z_loc="0.1" r_deg="-1.570795" p_deg="1.570795" y_deg="1.570795"/>
   </xacro:macro>
 </robot>

File: turtlebot_nonstop/turtlebot_nonstop_description/urdf/marker_bundle/marker_bundle_0.urdf.xacro (robot description, xacro)
@@ -38,8 +38,8 @@
   </xacro:macro>
   <xacro:macro name="marker_bundle_0" params="parent">
-    <attached_marker parent="${parent}" marker_num="0" direction="front" x_loc= "0.08" y_loc= "0.073" z_loc="0.253" r_deg="0" p_deg="1.570795" y_deg="0"/>
-    <attached_marker parent="${parent}" marker_num="1" direction="backward" x_loc= "-0.165" y_loc= "0" z_loc="0.253" r_deg="3.14159" p_deg="1.570795" y_deg="0"/>
-    <attached_marker parent="${parent}" marker_num="2" direction="left" x_loc="0" y_loc= "-0.17" z_loc="0.253" r_deg="3.14159" p_deg="1.570795" y_deg="1.570795"/>
-    <attached_marker parent="${parent}" marker_num="3" direction="right" x_loc= "0" y_loc="0.17" z_loc="0.253" r_deg="0" p_deg="1.570795" y_deg="1.570795"/>
+    <attached_marker parent="${parent}" marker_num="0" direction="front" x_loc= "-0.08" y_loc= "0.073" z_loc="0.253" r_deg="1.570795" p_deg="0" y_deg="1.570795"/>
+    <attached_marker parent="${parent}" marker_num="1" direction="backward" x_loc= "-0.165" y_loc= "0" z_loc="0.253" r_deg="1.570795" p_deg="0" y_deg="-1.570795"/>
+    <attached_marker parent="${parent}" marker_num="2" direction="left" x_loc="0" y_loc= "-0.17" z_loc="0.253" r_deg="1.570795" p_deg="0" y_deg="3.141592"/>
+    <attached_marker parent="${parent}" marker_num="3" direction="right" x_loc= "0" y_loc="0.17" z_loc="0.253" r_deg="1.570795" p_deg="0" y_deg="0"/>
       </xacro:macro>
 </robot>
